Commit message: go chase it 3

File: src/my_robot/urdf/my_robot.xacro (robot description, xacro)
@@ -58,5 +58,5 @@
     <inertial>
       <mass value="5.0"/>
-      <origin xyz="0.0 0 0" rpy="0 1.5707 1.5707"/>
+      <origin xyz="0 0 0" rpy="0 1.5707 1.5707"/>
       <inertia
           ixx="0.1" ixy="0" ixz="0"
@@ -110,5 +110,5 @@
   </joint>
  <joint type="continuous" name="right_wheel_hinge">
-    <origin xyz="0 0.15 0" rpy="0 0 0"/>
+    <origin xyz="0 -0.15 0" rpy="0 0 0"/>
     <child link="right_wheel"/>
     <parent link="chassis"/>
@@ -117,3 +117,53 @@
     <dynamics damping="1.0" friction="1.0"/>
   </joint>
+ <link name='camera'>
+ <pose>0 0 0 0 0 0<pose/>
+   <visual name='camera_visual'>
+     <geometry>
+        <box size="0.05 0.05 0.05"/>
+     </geometry>
+   </visual>
+   <collision name='camera_collision'>
+     <geometry>
+        <box size="0.05 0.05 0.05"/>
+     </geometry>
+   </collision>
+   <inertial>
+     <mass value="0.1"/>
+     <origin xyz="0.05 0.05 0.05" rpy="0 0 0"/>
+     <inertia
+        ixx="1e-6" ixy="0" ixz="0"
+        iyy="1e-6" iyz="0"
+        izz="1e-6"/>
+   </inertial>
+ </link>
+ <joint name='camera_joint' type='fixed'>
+  <origin xyz="0.2 0 0" rpy="0 0 0"/>
+  <parent link="chasis"/>
+  <child link="camera"/>
+  <axis xyz="0 1 0" rpy="0 0 0"/>
+ </joint>
+ <link name='hokuyo'>
+ <pose>0 0 0 0 0 0<pose/>
+   <visual name='hokuyo_visual'>
+     <geometry>
+        <mesh filename = "package://my_robot/meshes/hokuyo.dae"/>
+     </geometry>
+   </visual>
+   <collision>
+     <geometry>
+        <box size="0.1 0.1 0.1"/>
+     </geometry>
+   </collision>
+   <inertial name='hokuyo_inertial'>
+     <mass="1e-5"/>
+     <inertia ixx="1e-6" ixy="0" ixz="0" iyy="1e-6" iyz="0" izz="1e-6"/>
+   </inertial>
+ </link>
+ <joint name="hokuyo_joint" type="fixed">
+  <origin xyz="0.15 0 0.1" rpy="0 0 0"/>
+  <parent link="chasis"/>
+  <child link="hokuyo"/>
+  <axis xyz="0 1 0" rpy="0 0 0"/>
+ </joint>
 </robot>

Commit message: go chase it 4

File: src/my_robot/urdf/my_robot.xacro (robot description, xacro)
@@ -117,34 +117,36 @@
     <dynamics damping="1.0" friction="1.0"/>
   </joint>
- <link name='camera'>
- <pose>0 0 0 0 0 0<pose/>
-   <visual name='camera_visual'>
-     <geometry>
-        <box size="0.05 0.05 0.05"/>
-     </geometry>
-   </visual>
-   <collision name='camera_collision'>
-     <geometry>
-        <box size="0.05 0.05 0.05"/>
-     </geometry>
-   </collision>
-   <inertial>
-     <mass value="0.1"/>
-     <origin xyz="0.05 0.05 0.05" rpy="0 0 0"/>
-     <inertia
+  <link name='camera'>
+    <inertial>
+      <mass value="0.1"/>
+      <origin xyz="0.05 0.05 0.05" rpy="0 0 0" />
+      <inertia
         ixx="1e-6" ixy="0" ixz="0"
         iyy="1e-6" iyz="0"
-        izz="1e-6"/>
-   </inertial>
- </link>
- <joint name='camera_joint' type='fixed'>
-  <origin xyz="0.2 0 0" rpy="0 0 0"/>
-  <parent link="chasis"/>
-  <child link="camera"/>
-  <axis xyz="0 1 0" rpy="0 0 0"/>
- </joint>
+        izz="1e-6"
+      />
+    </inertial>
+    <collision name='camera_collision'>
+      <origin xyz="0 0 0" rpy="0 0 0"/>
+      <geometry>
+        <box size=".05 .05 .05"/>
+      </geometry>
+    </collision>
+    <visual name='camera_visual'>
+      <origin xyz="0 0 0" rpy="0 0 0"/>
+      <geometry>
+        <box size="0.05 0.05 0.05"/>
+      </geometry>
+    </visual>
+  </link>
+  <joint name='camera_joint' type='fixed'>
+    <origin xyz="0.2 0 0" rpy="0 0 0"/>
+    <parent link="chasis"/>
+    <child link="camera"/>
+    <axis xyz="0 1 0" />
+  </joint>
+<!--
  <link name='hokuyo'>
- <pose>0 0 0 0 0 0<pose/>
-   <visual name='hokuyo_visual'>
+    <visual name='hokuyo_visual'>
      <geometry>
         <mesh filename = "package://my_robot/meshes/hokuyo.dae"/>
@@ -157,5 +159,5 @@
    </collision>
    <inertial name='hokuyo_inertial'>
-     <mass="1e-5"/>
+     <mass value ="1e-5"/>
      <inertia ixx="1e-6" ixy="0" ixz="0" iyy="1e-6" iyz="0" izz="1e-6"/>
    </inertial>
@@ -167,3 +169,4 @@
   <axis xyz="0 1 0" rpy="0 0 0"/>
  </joint>
+-->
 </robot>

Commit message: go chase it 5

File: src/my_robot/urdf/my_robot.xacro (robot description, xacro)
@@ -2,4 +2,5 @@
 <robot name="my_robot" xmlns:xacro="http://www.ros.org/wiki/xacro">
   <link name="robot_footprint"></link>
+  <xacro:include filename="$(find my_robot)/urdf/my_robot.gazebo" />
   <joint name="robot_footprint_joint" type="fixed">
     <origin xyz="0 0 0" rpy="0 0 0" />
@@ -142,9 +143,8 @@
   <joint name='camera_joint' type='fixed'>
     <origin xyz="0.2 0 0" rpy="0 0 0"/>
-    <parent link="chasis"/>
+    <parent link="chassis"/>
     <child link="camera"/>
     <axis xyz="0 1 0" />
   </joint>
-<!--
  <link name='hokuyo'>
     <visual name='hokuyo_visual'>
@@ -165,8 +165,22 @@
  <joint name="hokuyo_joint" type="fixed">
   <origin xyz="0.15 0 0.1" rpy="0 0 0"/>
-  <parent link="chasis"/>
+  <parent link="chassis"/>
   <child link="hokuyo"/>
   <axis xyz="0 1 0" rpy="0 0 0"/>
  </joint>
--->
+  <gazebo reference ="left_wheel">
+    <material>Gazebo/Green</material>
+  </gazebo>
+   <gazebo reference ="right_wheel">
+    <material>Gazebo/Green</material>
+  </gazebo>
+   <gazebo reference ="robot_footprint">
+    <material>Gazebo/Black</material>
+  </gazebo>
+  <gazebo reference ="chassis">
+    <material>Gazebo/Blue</material>
+  </gazebo>
+  <gazebo reference ="camera">
+    <material>Gazebo/Red</material>
+  </gazebo>
 </robot>
